Commit message: dummy link established

File: abb_irb120_support/urdf/irb120_11.urdf (robot description, URDF)
Before this commit: robot abb_irb120_3_58, 10 links, 9 joints
Links:
- added link base_m
- added link flange_m
- added link link_1_m, mass 3.067; collision mesh filename=package://abb_irb120_support/meshes/irb120_3_58/collision/l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; visual mesh filename=package://abb_irb120_support/meshes/irb120_3_58/visual/link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
- added link link_2_m, mass 3.909; collision mesh filename=package://abb_irb120_support/meshes/irb120_3_58/collision/l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; visual mesh filename=package://abb_irb120_support/meshes/irb120_3_58/visual/link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
- added link link_3_m, mass 2.944; collision mesh filename=package://abb_irb120_support/meshes/irb120_3_58/collision/l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; visual mesh filename=package://abb_irb120_support/meshes/irb120_3_58/visual/link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
- added link link_4_m, mass 1.328; collision mesh filename=package://abb_irb120_support/meshes/irb120_3_58/collision/l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; visual mesh filename=package://abb_irb120_support/meshes/irb120_3_58/visual/link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
- added link link_5_m, mass 0.546; collision mesh filename=package://abb_irb120_support/meshes/irb120_3_58/collision/l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; visual mesh filename=package://abb_irb120_support/meshes/irb120_3_58/visual/link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
- added link link_6_m, mass 0.137; collision mesh filename=package://abb_irb120_support/meshes/irb120_3_58/collision/l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; visual mesh filename=package://abb_irb120_support/meshes/irb120_3_58/visual/link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
- added link tool0_m
Joints:
- added joint joint_1_m: type revolute, parent base_link, child link_1_m, origin xyz=1 0 0 rpy=0 0 0, axis 0 0 1, limit lower=-2.87979 upper=2.87979 effort=0 velocity=4.36332
- added joint joint_2_m: type revolute, parent link_1_m, child link_2_m, origin xyz=0 0 0.29 rpy=0 0 0, axis 0 1 0, limit lower=-1.91986 upper=1.91986 effort=0 velocity=4.36332
- added joint joint_3_m: type revolute, parent link_2_m, child link_3_m, origin xyz=0 0 0.27 rpy=0 0 0, axis 0 1 0, limit lower=-1.91986 upper=1.22173 effort=0 velocity=4.36332
- added joint joint_4_m: type revolute, parent link_3_m, child link_4_m, origin xyz=0 0 0.07 rpy=0 0 0, axis 1 0 0, limit lower=-2.79253 upper=2.79253 effort=0 velocity=5.58505
- added joint joint_5_m: type revolute, parent link_4_m, child link_5_m, origin xyz=0.302 0 0 rpy=0 0 0, axis 0 1 0, limit lower=-2.094395 upper=2.094395 effort=0 velocity=5.58505
- added joint joint_6_m: type revolute, parent link_5_m, child link_6_m, origin xyz=0.072 0 0 rpy=0 0 0, axis 1 0 0, limit lower=-6.98132 upper=6.98132 effort=0 velocity=7.33038
- added joint joint_6_m-flange_m: type fixed, parent link_6_m, child flange_m, origin xyz=0 0 0 rpy=0 0 0
- added joint link_6_m-tool0_m: type fixed, parent flange_m, child tool0_m, origin xyz=0 0 0 rpy=0 1.57079632679 0
- joint base_link-base: child base -> base_m

File: abb_irb120_support/urdf/irb120_3_58_macro.xacro (robot description, xacro)
@@ -4,4 +4,25 @@
   <xacro:macro name="abb_irb120_3_58" params="prefix">
     <!-- link list -->
+    <link name="${prefix}dummy">
+      <inertial>
+        <mass value="0"/>
+        <origin xyz="-0.04204 8.01E-05 0.07964" rpy="0 0 0"/>
+        <inertia ixx="0.0" ixy="0" ixz="0" iyy="0" iyz="0" izz="0"/>
+      </inertial>
+      <!--<visual>
+        <origin xyz="0.5 0 0" rpy="0 0 0"/>
+        <geometry>
+          <mesh filename="package://abb_irb120_support/meshes/irb120_3_58/visual/base_link.stl"/>
+        </geometry>
+        <xacro:material_abb_orange />
+      </visual>
+      <collision>
+        <origin xyz="0.5 0 0" rpy="0 0 0"/>
+        <geometry>
+          <mesh filename="package://abb_irb120_support/meshes/irb120_3_58/collision/base_link.stl"/>
+        </geometry>
+        <xacro:material_abb_yellow />
+      </collision> -->
+    </link>
     <link name="${prefix}base_link">
       <inertial>
@@ -152,4 +173,25 @@
     </link>
      <!-- mirror for second arm -->
+      <link name="${prefix}base_link_m">
+      <inertial>
+        <mass value="6.215"/>
+        <origin xyz="-0.04204 8.01E-05 0.07964" rpy="0 0 0"/>
+        <inertia ixx="0.0247272" ixy="-8.0784E-05" ixz="0.00130902" iyy="0.0491285" iyz="-8.0419E-06" izz="0.0472376"/>
+      </inertial>
+      <visual>
+        <origin xyz="1 0 0" rpy="0 0 3.14159"/>
+        <geometry>
+          <mesh filename="package://abb_irb120_support/meshes/irb120_3_58/visual/base_link.stl"/>
+        </geometry>
+        <xacro:material_abb_orange />
+      </visual>
+      <collision>
+        <origin xyz="1 0 0" rpy="0 0 3.14159"/>
+        <geometry>
+          <mesh filename="package://abb_irb120_support/meshes/irb120_3_58/collision/base_link.stl"/>
+        </geometry>
+        <xacro:material_abb_yellow />
+      </collision>
+    </link>
     <link name="${prefix}link_1_m">
       <inertial>
@@ -159,5 +201,5 @@
       </inertial>
       <visual>
-        <origin xyz="1 0 0" rpy="0 0 0"/>
+        <origin xyz="0 0 0" rpy="0 0 0"/>
         <geometry>
           <mesh filename="package://abb_irb120_support/meshes/irb120_3_58/visual/link_1.stl"/>
@@ -166,5 +208,5 @@
       </visual>
       <collision>
-        <origin xyz="1 0 0" rpy="0 0 0"/>
+        <origin xyz="0 0 0" rpy="0 0 0"/>
         <geometry>
           <mesh filename="package://abb_irb120_support/meshes/irb120_3_58/collision/link_1.stl"/>
@@ -180,5 +222,5 @@
       </inertial>
       <visual>
-        <origin xyz="1 0 0" rpy="0 0 0"/>
+        <origin xyz="0 0 0" rpy="0 0 0"/>
         <geometry>
           <mesh filename="package://abb_irb120_support/meshes/irb120_3_58/visual/link_2.stl"/>
@@ -187,5 +229,5 @@
       </visual>
       <collision>
-        <origin xyz="1 0 0" rpy="0 0 0"/>
+        <origin xyz="0 0 0" rpy="0 0 0"/>
         <geometry>
           <mesh filename="package://abb_irb120_support/meshes/irb120_3_58/collision/link_2.stl"/>
@@ -201,5 +243,5 @@
       </inertial>
       <visual>
-        <origin xyz="1 0 0" rpy="0 0 3.14159"/>
+        <origin xyz="0 0 0" rpy="0 0 3.14159"/>
         <geometry>
           <mesh filename="package://abb_irb120_support/meshes/irb120_3_58/visual/link_3.stl"/>
@@ -208,5 +250,5 @@
       </visual>
       <collision>
-        <origin xyz="1 0 0" rpy="0 0 3.14159"/>
+        <origin xyz="0 0 0" rpy="0 0 3.14159"/>
         <geometry>
           <mesh filename="package://abb_irb120_support/meshes/irb120_3_58/collision/link_3.stl"/>
@@ -222,5 +264,5 @@
       </inertial>
       <visual>
-        <origin xyz="1 0 0" rpy="0 3.14159 0"/>
+        <origin xyz="0 0 0" rpy="0 3.14159 0"/>
         <geometry>
           <mesh filename="package://abb_irb120_support/meshes/irb120_3_58/visual/link_4.stl"/>
@@ -229,5 +271,5 @@
       </visual>
       <collision>
-        <origin xyz="1 0 0" rpy="0 3.14159 0"/>
+        <origin xyz="0 0 0" rpy="0 3.14159 0"/>
         <geometry>
           <mesh filename="package://abb_irb120_support/meshes/irb120_3_58/collision/link_4.stl"/>
@@ -243,5 +285,5 @@
       </inertial>
       <visual>
-        <origin xyz="0.4 0 0" rpy="0 3.14159 0"/>
+        <origin xyz="-0.6 0 0" rpy="0 3.14159 0"/>
         <geometry>
           <mesh filename="package://abb_irb120_support/meshes/irb120_3_58/visual/link_5.stl"/>
@@ -250,5 +292,5 @@
       </visual>
       <collision>
-        <origin xyz="0.4 0 0" rpy="0 3.14159 0"/>
+        <origin xyz="-0.6 0 0" rpy="0 3.14159 0"/>
         <geometry>
           <mesh filename="package://abb_irb120_support/meshes/irb120_3_58/collision/link_5.stl"/>
@@ -264,5 +306,5 @@
       </inertial>
       <visual>
-        <origin xyz="0.4 0 0" rpy="0 3.14159 0"/>
+        <origin xyz="-0.6 0 0" rpy="0 3.14159 0"/>
         <geometry>
           <mesh filename="package://abb_irb120_support/meshes/irb120_3_58/visual/link_6.stl"/>
@@ -271,5 +313,5 @@
       </visual>
       <collision>
-        <origin xyz="0.4 0 0" rpy="0 3.14159 0"/>
+        <origin xyz="-0.6 0 0" rpy="0 3.14159 0"/>
         <geometry>
           <mesh filename="package://abb_irb120_support/meshes/irb120_3_58/collision/link_6.stl"/>
@@ -281,4 +323,12 @@
     <!-- joint list -->
     <joint name="${prefix}joint_1" type="revolute">
+      <origin rpy="0 0 0" xyz="0 0 0"/>
+      <parent link="${prefix}dummy"/>
+      <child link="${prefix}base_link"/>
+      <limit effort="0" lower="-2.87979" upper="2.87979" velocity="4.36332"/>
+      <axis xyz="0 0 1"/>
+      <dynamics damping="0.0" friction="0.0"/>
+    </joint>
+    <joint name="${prefix}joint_2" type="revolute">
       <origin rpy="0 0 0" xyz="0 0 0"/>
       <parent link="${prefix}base_link"/>
@@ -288,5 +338,5 @@
       <dynamics damping="0.0" friction="0.0"/>
     </joint>
-    <joint name="${prefix}joint_2" type="revolute">
+    <joint name="${prefix}joint_3" type="revolute">
       <origin rpy="0 0 0" xyz="0 0 0.29"/>
       <parent link="${prefix}link_1"/>
@@ -296,5 +346,5 @@
       <dynamics damping="0.0" friction="0.0"/>
     </joint>
-    <joint name="${prefix}joint_3" type="revolute">
+    <joint name="${prefix}joint_4" type="revolute">
       <origin rpy="0 0 0" xyz="0 0 0.27"/>
       <parent link="${prefix}link_2"/>
@@ -304,5 +354,5 @@
       <dynamics damping="0.0" friction="0.0"/>
     </joint>
-    <joint name="${prefix}joint_4" type="revolute">
+    <joint name="${prefix}joint_5" type="revolute">
       <origin rpy="0 0 0" xyz="0 0 0.07"/>
       <parent link="${prefix}link_3"/>
@@ -312,5 +362,5 @@
       <dynamics damping="0.0" friction="0.0"/>
     </joint>
-    <joint name="${prefix}joint_5" type="revolute">
+    <joint name="${prefix}joint_6" type="revolute">
       <origin rpy="0 0 0" xyz="0.302 0 0"/>
       <parent link="${prefix}link_4"/>
@@ -320,5 +370,5 @@
       <dynamics damping="0.0" friction="0.0"/>
     </joint>
-    <joint name="${prefix}joint_6" type="revolute">
+    <joint name="${prefix}joint_7" type="revolute">
       <origin rpy="0 0 0" xyz="0.072 0 0"/>
       <parent link="${prefix}link_5"/>
@@ -331,5 +381,13 @@
     <joint name="${prefix}joint_1_m" type="revolute">
       <origin rpy="0 0 0" xyz="1 0 0"/>
-      <parent link="${prefix}base_link"/>
+      <parent link="${prefix}dummy"/>
+      <child link="${prefix}base_link_m"/>
+      <limit effort="0" lower="-2.87979" upper="2.87979" velocity="4.36332"/>
+      <axis xyz="0 0 1"/>
+      <dynamics damping="0.0" friction="0.0"/>
+    </joint>
+    <joint name="${prefix}joint_2_m" type="revolute">
+      <origin rpy="0 0 0" xyz="1 0 0"/>
+      <parent link="${prefix}base_link_m"/>
       <child link="${prefix}link_1_m"/>
       <limit effort="0" lower="-2.87979" upper="2.87979" velocity="4.36332"/>
@@ -337,5 +395,5 @@
       <dynamics damping="0.0" friction="0.0"/>
     </joint>
-    <joint name="${prefix}joint_2_m" type="revolute">
+    <joint name="${prefix}joint_3_m" type="revolute">
       <origin rpy="0 0 0" xyz="0 0 0.29"/>
       <parent link="${prefix}link_1_m"/>
@@ -345,5 +403,5 @@
       <dynamics damping="0.0" friction="0.0"/>
     </joint>
-    <joint name="${prefix}joint_3_m" type="revolute">
+    <joint name="${prefix}joint_4_m" type="revolute">
       <origin rpy="0 0 0" xyz="0 0 0.27"/>
       <parent link="${prefix}link_2_m"/>
@@ -353,5 +411,5 @@
       <dynamics damping="0.0" friction="0.0"/>
     </joint>
-    <joint name="${prefix}joint_4_m" type="revolute">
+    <joint name="${prefix}joint_5_m" type="revolute">
       <origin rpy="0 0 0" xyz="0 0 0.07"/>
       <parent link="${prefix}link_3_m"/>
@@ -361,5 +419,5 @@
       <dynamics damping="0.0" friction="0.0"/>
     </joint>
-    <joint name="${prefix}joint_5_m" type="revolute">
+    <joint name="${prefix}joint_6_m" type="revolute">
       <origin rpy="0 0 0" xyz="0.302 0 0"/>
       <parent link="${prefix}link_4_m"/>
@@ -369,5 +427,5 @@
       <dynamics damping="0.0" friction="0.0"/>
     </joint>
-    <joint name="${prefix}joint_6_m" type="revolute">
+    <joint name="${prefix}joint_7_m" type="revolute">
       <origin rpy="0 0 0" xyz="0.072 0 0"/>
       <parent link="${prefix}link_5_m"/>
@@ -380,7 +438,7 @@
     <!-- ROS-Industrial 'base' frame: base_link to ABB World Coordinates transform -->
     <link name="${prefix}base" />
-    <joint name="${prefix}base_link-base" type="fixed">
+    <joint name="${prefix}dummy-base" type="fixed">
       <origin xyz="0 0 0" rpy="0 0 0"/>
-      <parent link="${prefix}base_link"/>
+      <parent link="${prefix}dummy"/>
       <child link="${prefix}base"/>
     </joint>

File: abb_irb120_support/urdf/irb_120_12.urdf (robot description, URDF)
Before this commit: robot abb_irb120_3_58, 16 links, 15 joints
Links:
- added link base_link_m, mass 6.215; collision mesh filename=package://abb_irb120_support/meshes/irb120_3_58/collision/b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; visual mesh filename=package://abb_irb120_support/meshes/irb120_3_58/visual/base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
- added link dummy, mass 6.215; collision mesh filename=package://abb_irb120_support/meshes/irb120_3_58/collision/b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; visual mesh filename=package://abb_irb120_support/meshes/irb120_3_58/visual/base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
- added link flange_m
- added link tool0_m
Joints:
- removed joint base_link-base
- added joint dummy-base: type fixed, parent dummy, child base, origin xyz=0 0 0 rpy=0 0 0
- added joint joint_6_m-flange_m: type fixed, parent link_6_m, child flange_m, origin xyz=0 0 0 rpy=0 0 0
- added joint link_6_m-tool0_m: type fixed, parent flange_m, child tool0_m, origin xyz=0 0 0 rpy=0 1.57079632679 0
- joint joint_1_m: parent base_link -> base_link_m
- joint joint_2_m: origin xyz=1 0 0.29 rpy=0 0 0 -> xyz=0 0 0.29 rpy=0 0 0
- joint joint_3_m: origin xyz=1 0 0.27 rpy=0 0 0 -> xyz=0 0 0.27 rpy=0 0 0
- joint joint_4_m: origin xyz=1 0 0.07 rpy=0 0 0 -> xyz=0 0 0.07 rpy=0 0 0
- joint joint_5_m: origin xyz=1.302 0 0 rpy=0 0 0 -> xyz=0.302 0 0 rpy=0 0 0
- joint joint_6_m: origin xyz=1.072 0 0 rpy=0 0 0 -> xyz=0.072 0 0 rpy=0 0 0

File: abb_irb120_support/urdf/irb_120_14.urdf (robot description, URDF)
Before this commit: robot abb_irb120_3_58, 18 links, 17 joints
Links:
- added link base_link_m, mass 6.215; collision mesh filename=package://abb_irb120_support/meshes/irb120_3_58/collision/b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; visual mesh filename=package://abb_irb120_support/meshes/irb120_3_58/visual/base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
- added link dummy, mass 6.215; collision mesh filename=package://abb_irb120_support/meshes/irb120_3_58/collision/b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; visual mesh filename=package://abb_irb120_support/meshes/irb120_3_58/visual/base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
Joints:
- removed joint base_link-base
- added joint dummy-base: type fixed, parent dummy, child base, origin xyz=0 0 0 rpy=0 0 0
- added joint joint_7: type revolute, parent link_5, child link_6, origin xyz=0.072 0 0 rpy=0 0 0, axis 1 0 0, limit lower=-6.98132 upper=6.98132 effort=0 velocity=7.33038
- added joint joint_7_m: type revolute, parent link_5_m, child link_6_m, origin xyz=0.072 0 0 rpy=0 0 0, axis 1 0 0, limit lower=-6.98132 upper=6.98132 effort=0 velocity=7.33038
- joint joint_1: child link_1 -> base_link; parent base_link -> dummy
- joint joint_1_m: child link_1_m -> base_link_m; parent base_link -> dummy
- joint joint_2: axis 0 1 0 -> 0 0 1; child link_2 -> link_1; limit lower=-1.91986 upper=1.91986 effort=0 velocity=4.36332 -> lower=-2.87979 upper=2.87979 effort=0 velocity=4.36332; origin xyz=0 0 0.29 rpy=0 0 0 -> xyz=0 0 0 rpy=0 0 0; parent link_1 -> base_link
- joint joint_2_m: axis 0 1 0 -> 0 0 1; child link_2_m -> link_1_m; limit lower=-1.91986 upper=1.91986 effort=0 velocity=4.36332 -> lower=-2.87979 upper=2.87979 effort=0 velocity=4.36332; origin xyz=0 0 0.29 rpy=0 0 0 -> xyz=1 0 0 rpy=0 0 0; parent link_1_m -> base_link_m
- joint joint_3: child link_3 -> link_2; limit lower=-1.91986 upper=1.22173 effort=0 velocity=4.36332 -> lower=-1.91986 upper=1.91986 effort=0 velocity=4.36332; origin xyz=0 0 0.27 rpy=0 0 0 -> xyz=0 0 0.29 rpy=0 0 0; parent link_2 -> link_1
- joint joint_3_m: child link_3_m -> link_2_m; limit lower=-1.91986 upper=1.22173 effort=0 velocity=4.36332 -> lower=-1.91986 upper=1.91986 effort=0 velocity=4.36332; origin xyz=0 0 0.27 rpy=0 0 0 -> xyz=0 0 0.29 rpy=0 0 0; parent link_2_m -> link_1_m
- joint joint_4: axis 1 0 0 -> 0 1 0; child link_4 -> link_3; limit lower=-2.79253 upper=2.79253 effort=0 velocity=5.58505 -> lower=-1.91986 upper=1.22173 effort=0 velocity=4.36332; origin xyz=0 0 0.07 rpy=0 0 0 -> xyz=0 0 0.27 rpy=0 0 0; parent link_3 -> link_2
- joint joint_4_m: axis 1 0 0 -> 0 1 0; child link_4_m -> link_3_m; limit lower=-2.79253 upper=2.79253 effort=0 velocity=5.58505 -> lower=-1.91986 upper=1.22173 effort=0 velocity=4.36332; origin xyz=0 0 0.07 rpy=0 0 0 -> xyz=0 0 0.27 rpy=0 0 0; parent link_3_m -> link_2_m
- joint joint_5: axis 0 1 0 -> 1 0 0; child link_5 -> link_4; limit lower=-2.094395 upper=2.094395 effort=0 velocity=5.58505 -> lower=-2.79253 upper=2.79253 effort=0 velocity=5.58505; origin xyz=0.302 0 0 rpy=0 0 0 -> xyz=0 0 0.07 rpy=0 0 0; parent link_4 -> link_3
- joint joint_5_m: axis 0 1 0 -> 1 0 0; child link_5_m -> link_4_m; limit lower=-2.094395 upper=2.094395 effort=0 velocity=5.58505 -> lower=-2.79253 upper=2.79253 effort=0 velocity=5.58505; origin xyz=0.302 0 0 rpy=0 0 0 -> xyz=0 0 0.07 rpy=0 0 0; parent link_4_m -> link_3_m
- joint joint_6: axis 1 0 0 -> 0 1 0; child link_6 -> link_5; limit lower=-6.98132 upper=6.98132 effort=0 velocity=7.33038 -> lower=-2.094395 upper=2.094395 effort=0 velocity=5.58505; origin xyz=0.072 0 0 rpy=0 0 0 -> xyz=0.302 0 0 rpy=0 0 0; parent link_5 -> link_4
- joint joint_6_m: axis 1 0 0 -> 0 1 0; child link_6_m -> link_5_m; limit lower=-6.98132 upper=6.98132 effort=0 velocity=7.33038 -> lower=-2.094395 upper=2.094395 effort=0 velocity=5.58505; origin xyz=0.072 0 0 rpy=0 0 0 -> xyz=0.302 0 0 rpy=0 0 0; parent link_5_m -> link_4_m
