Commit message: working on joints with joint_state_publisher

File: abb_irb120_support/urdf/irb120_3_58_macro_revert.xacro (robot description, xacro)
@@ -448,5 +448,5 @@
     <!-- ROS-Industrial 'flange' frame: attachment point for EEF models -->
     <link name="${prefix}flange"/>
-    <joint type="fixed" name="${prefix}joint_8-flange">
+    <joint type="fixed" name="${prefix}joint_6-flange">
       <origin xyz="0 0 0" rpy="0 0 0"/>
       <parent link="${prefix}link_6"/>
@@ -455,5 +455,5 @@
     <!-- mirror -->
     <link name="${prefix}flange_m"/>
-    <joint type="fixed" name="${prefix}joint_8_m-flange_m">
+    <joint type="fixed" name="${prefix}joint_6_m-flange_m">
       <origin xyz="0 0 0" rpy="0 0 0"/>
       <parent link="${prefix}link_6_m"/>
@@ -462,5 +462,5 @@
     <!-- ROS-Industrial 'tool0' frame: all-zeros tool frame -->
     <link name="${prefix}tool0" />
-    <joint name="${prefix}link_7-tool0" type="fixed">
+    <joint name="${prefix}link_6-tool0" type="fixed">
       <origin xyz="0 0 0" rpy="0 ${radians(90)} 0" />
       <parent link="${prefix}flange" />
@@ -469,5 +469,5 @@
     <!-- mirror -->
     <link name="${prefix}tool0_m" />
-    <joint name="${prefix}link_7_m-tool0_m" type="fixed">
+    <joint name="${prefix}link_6_m-tool0_m" type="fixed">
       <origin xyz="0 0 0" rpy="0 ${radians(90)} 0" />
       <parent link="${prefix}flange_m" />
