Commit message: dual arm - working

File: abb_irb120_support/urdf/irb120_3_58_macro_revert_1.xacro (robot description, xacro)
@@ -192,5 +192,5 @@
       </inertial>
       <visual>
-        <origin xyz="0 0 0" rpy="0 0 3.14159"/>
+        <origin xyz="0 0 0" rpy="0 0 0"/>
         <geometry>
           <mesh filename="package://abb_irb120_support/meshes/irb120_3_58/visual/link_1.stl"/>
@@ -199,5 +199,5 @@
       </visual>
       <collision>
-        <origin xyz="0 0 0" rpy="0 0 3.14159"/>
+        <origin xyz="0 0 0" rpy="0 0 0"/>
         <geometry>
           <mesh filename="package://abb_irb120_support/meshes/irb120_3_58/collision/link_1.stl"/>
@@ -251,9 +251,9 @@
       <inertial>
         <mass value="1.328"/>
-        <origin xyz="2.2247 0.00015 0.00041" rpy="0 0 0"/>
+        <origin xyz="0.2247 0.00015 0.00041" rpy="0 0 0"/>
         <inertia ixx="0.00284661" ixy="-2.12765E-05" ixz="-1.6435E-05" iyy="0.00401346" iyz="1.31336E-05" izz="0.0052535"/>
       </inertial>
       <visual>
-        <origin xyz="0 0 0" rpy="3.14159 3.14159 0"/>
+        <origin xyz="0 0 0" rpy="0 3.14159 0"/>
         <geometry>
           <mesh filename="package://abb_irb120_support/meshes/irb120_3_58/visual/link_4.stl"/>
@@ -262,5 +262,5 @@
       </visual>
       <collision>
-        <origin xyz="0 0 0" rpy="3.14159 3.14159 0"/>
+        <origin xyz="0 0 0" rpy="0 3.14159 0"/>
         <geometry>
           <mesh filename="package://abb_irb120_support/meshes/irb120_3_58/collision/link_4.stl"/>
@@ -272,9 +272,9 @@
       <inertial>
         <mass value="0.546"/>
-        <origin xyz="-0.60109 3.68E-05 6.22E-05" rpy="0 0 0"/>
+        <origin xyz="-0.00109 3.68E-05 6.22E-05" rpy="0 0 0"/>
         <inertia ixx="0.000404891" ixy="1.61943E-06" ixz="8.46805E-07" iyy="0.000892825" iyz="-1.51792E-08" izz="0.000815468"/>
       </inertial>
       <visual>
-        <origin xyz="0 0 0" rpy="0 3.14159 0"/>
+        <origin xyz="-0.6 0 0" rpy="0 3.14159 0"/>
         <geometry>
           <mesh filename="package://abb_irb120_support/meshes/irb120_3_58/visual/link_5.stl"/>
@@ -283,5 +283,5 @@
       </visual>
       <collision>
-        <origin xyz="0 0 0" rpy="0 3.14159 0"/>
+        <origin xyz="-0.6 0 0" rpy="0 3.14159 0"/>
         <geometry>
           <mesh filename="package://abb_irb120_support/meshes/irb120_3_58/collision/link_5.stl"/>
@@ -297,5 +297,5 @@
       </inertial>
       <visual>
-        <origin xyz="0 0 0" rpy="0 3.14159 0"/>
+        <origin xyz="-0.745 0 0" rpy="0 3.14159 0"/>
         <geometry>
           <mesh filename="package://abb_irb120_support/meshes/irb120_3_58/visual/link_6.stl"/>
@@ -304,5 +304,5 @@
       </visual>
       <collision>
-        <origin xyz="0 0 0" rpy="0 3.14159 0"/>
+        <origin xyz="-0.745 0 0" rpy="0 3.14159 0"/>
         <geometry>
           <mesh filename="package://abb_irb120_support/meshes/irb120_3_58/collision/link_6.stl"/>
@@ -312,5 +312,5 @@
     </link>
     <!-- end of link list -->
-    <!-- joint list
+    <!-- joint list -->
     <joint name="${prefix}joint_1" type="revolute">
       <origin rpy="0 0 0" xyz="0.5 0 0"/>
@@ -320,5 +320,5 @@
       <axis xyz="0 0 1"/>
       <dynamics damping="0.0" friction="0.0"/>
-    </joint> -->
+    </joint>
     <joint name="${prefix}joint_2" type="revolute">
       <origin rpy="0 0 0" xyz="0 0 0"/>
@@ -369,5 +369,5 @@
       <dynamics damping="0.0" friction="0.0"/>
     </joint>
-    <!-- joint list - mirror
+    <!-- joint list - mirror -->
     <joint name="${prefix}joint_1_m" type="revolute">
       <origin rpy="0 0 0" xyz="1.5 0 0"/>
@@ -377,5 +377,5 @@
       <axis xyz="0 0 1"/>
       <dynamics damping="0.0" friction="0.0"/>
-    </joint> -->
+    </joint>
     <joint name="${prefix}joint_2_m" type="revolute">
       <origin rpy="0 0 0" xyz="1 0 0"/>
@@ -411,5 +411,5 @@
     </joint>
     <joint name="${prefix}joint_6_m" type="revolute">
-      <origin rpy="0 0 0" xyz="-0.302 0 0"/>
+      <origin rpy="0 0 0" xyz="0.302 0 0"/>
       <parent link="${prefix}link_4_m"/>
       <child link="${prefix}link_5_m"/>
@@ -419,5 +419,5 @@
     </joint>
     <joint name="${prefix}joint_7_m" type="revolute">
-      <origin rpy="0 0 0" xyz="-0.072 0 0"/>
+      <origin rpy="0 0 0" xyz="0.072 0 0"/>
       <parent link="${prefix}link_5_m"/>
       <child link="${prefix}link_6_m"/>
@@ -433,14 +433,4 @@
       <parent link="${prefix}dummy"/>
       <child link="${prefix}base"/>
-    </joint>
-    <joint name="${prefix}dummy-base_link" type="fixed">
-      <origin xyz="0 0 0" rpy="0 0 0"/>
-      <parent link="${prefix}dummy"/>
-      <child link="${prefix}base_link"/>
-    </joint>
-    <joint name="${prefix}dummy-base_link_m" type="fixed">
-      <origin xyz="0 0 0" rpy="0 0 0"/>
-      <parent link="${prefix}dummy"/>
-      <child link="${prefix}base_link_m"/>
     </joint>
     <!--<link name="${prefix}base_1" />
@@ -480,5 +470,5 @@
     <link name="${prefix}tool0_m" />
     <joint name="${prefix}link_7_m-tool0_m" type="fixed">
-      <origin xyz="-0.01 0 0" rpy="0 ${radians(90)} 0" />
+      <origin xyz="0 0 0" rpy="0 ${radians(90)} 0" />
       <parent link="${prefix}flange_m" />
       <child link="${prefix}tool0_m" />
