Commit message: two arm urdf - done

File: abb_irb120_support/urdf/irb120_3_58_macro.xacro (robot description, xacro)
@@ -145,4 +145,131 @@
       <collision>
         <origin xyz="0 0 0" rpy="0 0 0"/>
+        <geometry>
+          <mesh filename="package://abb_irb120_support/meshes/irb120_3_58/collision/link_6.stl"/>
+        </geometry>
+        <xacro:material_abb_yellow />
+      </collision>
+    </link>
+     <!-- mirror for second arm -->
+    <link name="${prefix}link_1_m">
+      <inertial>
+        <mass value="3.067" />
+        <origin xyz="9.77E-05 -0.00012 0.23841" rpy="0 0 0"/>
+        <inertia ixx="0.0142175" ixy="-1.28579E-05" ixz="-2.31364E-05" iyy="0.0144041" iyz="1.93404E-05" izz="0.0104533"/>
+      </inertial>
+      <visual>
+        <origin xyz="1 0 0" rpy="0 0 0"/>
+        <geometry>
+          <mesh filename="package://abb_irb120_support/meshes/irb120_3_58/visual/link_1.stl"/>
+        </geometry>
+        <xacro:material_abb_orange />
+      </visual>
+      <collision>
+        <origin xyz="1 0 0" rpy="0 0 0"/>
+        <geometry>
+          <mesh filename="package://abb_irb120_support/meshes/irb120_3_58/collision/link_1.stl"/>
+        </geometry>
+        <xacro:material_abb_yellow />
+      </collision>
+    </link>
+    <link name="${prefix}link_2_m">
+      <inertial>
+        <mass value="3.909"/>
+        <origin xyz="0.00078 -0.00212 0.10124" rpy="0 0 0"/>
+        <inertia ixx="0.0603111" ixy="9.83431E-06" ixz="5.72407E-05" iyy="0.041569" iyz="-0.00050497" izz="0.0259548"/>
+      </inertial>
+      <visual>
+        <origin xyz="1 0 0" rpy="0 0 0"/>
+        <geometry>
+          <mesh filename="package://abb_irb120_support/meshes/irb120_3_58/visual/link_2.stl"/>
+        </geometry>
+        <xacro:material_abb_orange />
+      </visual>
+      <collision>
+        <origin xyz="1 0 0" rpy="0 0 0"/>
+        <geometry>
+          <mesh filename="package://abb_irb120_support/meshes/irb120_3_58/collision/link_2.stl"/>
+        </geometry>
+        <xacro:material_abb_yellow />
+      </collision>
+    </link>
+    <link name="${prefix}link_3_m">
+      <inertial>
+        <mass value="2.944"/>
+        <origin xyz="0.02281 0.00106 0.05791" rpy="0 0 0"/>
+        <inertia ixx="0.00835606" ixy="-8.01545E-05" ixz="0.00142884" iyy="0.016713" iyz="-0.000182227" izz="0.0126984"/>
+      </inertial>
+      <visual>
+        <origin xyz="1 0 0" rpy="0 0 3.14159"/>
+        <geometry>
+          <mesh filename="package://abb_irb120_support/meshes/irb120_3_58/visual/link_3.stl"/>
+        </geometry>
+        <xacro:material_abb_orange />
+      </visual>
+      <collision>
+        <origin xyz="1 0 0" rpy="0 0 3.14159"/>
+        <geometry>
+          <mesh filename="package://abb_irb120_support/meshes/irb120_3_58/collision/link_3.stl"/>
+        </geometry>
+        <xacro:material_abb_yellow />
+      </collision>
+    </link>
+    <link name="${prefix}link_4_m">
+      <inertial>
+        <mass value="1.328"/>
+        <origin xyz="0.2247 0.00015 0.00041" rpy="0 0 0"/>
+        <inertia ixx="0.00284661" ixy="-2.12765E-05" ixz="-1.6435E-05" iyy="0.00401346" iyz="1.31336E-05" izz="0.0052535"/>
+      </inertial>
+      <visual>
+        <origin xyz="1 0 0" rpy="0 3.14159 0"/>
+        <geometry>
+          <mesh filename="package://abb_irb120_support/meshes/irb120_3_58/visual/link_4.stl"/>
+        </geometry>
+        <xacro:material_abb_orange />
+      </visual>
+      <collision>
+        <origin xyz="1 0 0" rpy="0 3.14159 0"/>
+        <geometry>
+          <mesh filename="package://abb_irb120_support/meshes/irb120_3_58/collision/link_4.stl"/>
+        </geometry>
+        <xacro:material_abb_yellow />
+      </collision>
+    </link>
+    <link name="${prefix}link_5_m">
+      <inertial>
+        <mass value="0.546"/>
+        <origin xyz="-0.00109 3.68E-05 6.22E-05" rpy="0 0 0"/>
+        <inertia ixx="0.000404891" ixy="1.61943E-06" ixz="8.46805E-07" iyy="0.000892825" iyz="-1.51792E-08" izz="0.000815468"/>
+      </inertial>
+      <visual>
+        <origin xyz="0.4 0 0" rpy="0 3.14159 0"/>
+        <geometry>
+          <mesh filename="package://abb_irb120_support/meshes/irb120_3_58/visual/link_5.stl"/>
+        </geometry>
+        <xacro:material_abb_orange />
+      </visual>
+      <collision>
+        <origin xyz="0.4 0 0" rpy="0 3.14159 0"/>
+        <geometry>
+          <mesh filename="package://abb_irb120_support/meshes/irb120_3_58/collision/link_5.stl"/>
+        </geometry>
+        <xacro:material_abb_yellow />
+      </collision>
+    </link>
+    <link name="${prefix}link_6_m">
+      <inertial>
+        <mass value="0.137"/>
+        <origin xyz="-0.00706 -0.00017 -1.32E-06" rpy="0 0 0"/>
+        <inertia ixx="0.001" ixy="0" ixz="0" iyy="0.001" iyz="0" izz="0.001"/>
+      </inertial>
+      <visual>
+        <origin xyz="0.4 0 0" rpy="0 3.14159 0"/>
+        <geometry>
+          <mesh filename="package://abb_irb120_support/meshes/irb120_3_58/visual/link_6.stl"/>
+        </geometry>
+        <xacro:material_abb_black />
+      </visual>
+      <collision>
+        <origin xyz="0.4 0 0" rpy="0 3.14159 0"/>
         <geometry>
           <mesh filename="package://abb_irb120_support/meshes/irb120_3_58/collision/link_6.stl"/>
@@ -201,4 +328,53 @@
       <dynamics damping="0.0" friction="0.0"/>
     </joint>
+    <!-- joint list - mirror -->
+    <joint name="${prefix}joint_1_m" type="revolute">
+      <origin rpy="0 0 0" xyz="1 0 0"/>
+      <parent link="${prefix}base_link"/>
+      <child link="${prefix}link_1_m"/>
+      <limit effort="0" lower="-2.87979" upper="2.87979" velocity="4.36332"/>
+      <axis xyz="0 0 1"/>
+      <dynamics damping="0.0" friction="0.0"/>
+    </joint>
+    <joint name="${prefix}joint_2_m" type="revolute">
+      <origin rpy="0 0 0" xyz="0 0 0.29"/>
+      <parent link="${prefix}link_1_m"/>
+      <child link="${prefix}link_2_m"/>
+      <limit effort="0" lower="-1.91986" upper="1.91986" velocity="4.36332"/>
+      <axis xyz="0 1 0"/>
+      <dynamics damping="0.0" friction="0.0"/>
+    </joint>
+    <joint name="${prefix}joint_3_m" type="revolute">
+      <origin rpy="0 0 0" xyz="0 0 0.27"/>
+      <parent link="${prefix}link_2_m"/>
+      <child link="${prefix}link_3_m"/>
+      <limit effort="0" lower="-1.91986" upper="1.22173" velocity="4.36332"/>
+      <axis xyz="0 1 0"/>
+      <dynamics damping="0.0" friction="0.0"/>
+    </joint>
+    <joint name="${prefix}joint_4_m" type="revolute">
+      <origin rpy="0 0 0" xyz="0 0 0.07"/>
+      <parent link="${prefix}link_3_m"/>
+      <child link="${prefix}link_4_m"/>
+      <limit effort="0" lower="-2.79253" upper="2.79253" velocity="5.58505"/>
+      <axis xyz="1 0 0"/>
+      <dynamics damping="0.0" friction="0.0"/>
+    </joint>
+    <joint name="${prefix}joint_5_m" type="revolute">
+      <origin rpy="0 0 0" xyz="0.302 0 0"/>
+      <parent link="${prefix}link_4_m"/>
+      <child link="${prefix}link_5_m"/>
+      <limit effort="0" lower="-2.094395" upper="2.094395" velocity="5.58505"/>
+      <axis xyz="0 1 0"/>
+      <dynamics damping="0.0" friction="0.0"/>
+    </joint>
+    <joint name="${prefix}joint_6_m" type="revolute">
+      <origin rpy="0 0 0" xyz="0.072 0 0"/>
+      <parent link="${prefix}link_5_m"/>
+      <child link="${prefix}link_6_m"/>
+      <limit effort="0" lower="-6.98132" upper="6.98132" velocity="7.33038"/>
+      <axis xyz="1 0 0"/>
+      <dynamics damping="0.0" friction="0.0"/>
+    </joint>
     <!-- end of joint list -->
     <!-- ROS-Industrial 'base' frame: base_link to ABB World Coordinates transform -->

Commit message: collision solved + common root link established

File: abb_irb120_support/urdf/irb120_3_58_macro.xacro (robot description, xacro)
@@ -392,4 +392,11 @@
       <child link="${prefix}flange"/>
     </joint>
+    <!-- mirror -->
+    <link name="${prefix}flange_m"/>
+    <joint type="fixed" name="${prefix}joint_6_m-flange_m">
+      <origin xyz="0 0 0" rpy="0 0 0"/>
+      <parent link="${prefix}link_6_m"/>
+      <child link="${prefix}flange_m"/>
+    </joint>
     <!-- ROS-Industrial 'tool0' frame: all-zeros tool frame -->
     <link name="${prefix}tool0" />
@@ -399,4 +406,11 @@
       <child link="${prefix}tool0" />
     </joint>
+    <!-- mirror -->
+    <link name="${prefix}tool0_m" />
+    <joint name="${prefix}link_6_m-tool0_m" type="fixed">
+      <origin xyz="0 0 0" rpy="0 ${radians(90)} 0" />
+      <parent link="${prefix}flange_m" />
+      <child link="${prefix}tool0_m" />
+    </joint>
   </xacro:macro>
 </robot>

Commit message: added group states

File: abb_irb120_support/urdf/irb120_3_58_macro.xacro (robot description, xacro)
@@ -443,4 +443,16 @@
       <child link="${prefix}base"/>
     </joint>
+    <!--<link name="${prefix}base_1" />
+    <joint name="${prefix}base_link-base" type="fixed">
+      <origin xyz="0 0 0" rpy="0 0 0"/>
+      <parent link="${prefix}base"/>
+      <child link="${prefix}base_link"/>
+    </joint>
+    <link name="${prefix}base_m" />
+    <joint name="${prefix}base_link-base" type="fixed">
+      <origin xyz="0 0 0" rpy="0 0 0"/>
+      <parent link="${prefix}base"/>
+      <child link="${prefix}base_link_m"/>
+    </joint> -->
     <!-- ROS-Industrial 'flange' frame: attachment point for EEF models -->
     <link name="${prefix}flange"/>

Commit message: dual arm - in progress

File: abb_irb120_support/urdf/irb120_3_58_macro.xacro (robot description, xacro)
@@ -5,17 +5,8 @@
     <!-- link list -->
     <link name="${prefix}dummy">
-      <inertial>
-        <mass value="0"/>
-        <origin xyz="-0.04204 8.01E-05 0.07964" rpy="0 0 0"/>
-        <inertia ixx="0.0" ixy="0" ixz="0" iyy="0" iyz="0" izz="0"/>
-      </inertial>
-      <!--<visual>
+      <visual>
         <origin xyz="0.5 0 0" rpy="0 0 0"/>
-        <geometry>
-          <mesh filename="package://abb_irb120_support/meshes/irb120_3_58/visual/base_link.stl"/>
-        </geometry>
-        <xacro:material_abb_orange />
-      </visual>
-      <collision>
+      </visual>
+      <!--<collision>
         <origin xyz="0.5 0 0" rpy="0 0 0"/>
         <geometry>
@@ -323,5 +314,5 @@
     <!-- joint list -->
     <joint name="${prefix}joint_1" type="revolute">
-      <origin rpy="0 0 0" xyz="0 0 0"/>
+      <origin rpy="0 0 0" xyz="0.5 0 0"/>
       <parent link="${prefix}dummy"/>
       <child link="${prefix}base_link"/>
@@ -380,5 +371,5 @@
     <!-- joint list - mirror -->
     <joint name="${prefix}joint_1_m" type="revolute">
-      <origin rpy="0 0 0" xyz="1 0 0"/>
+      <origin rpy="0 0 0" xyz="1.5 0 0"/>
       <parent link="${prefix}dummy"/>
       <child link="${prefix}base_link_m"/>

Commit message: interactive marker size change

File: abb_irb120_support/urdf/irb120_3_58_macro.xacro (robot description, xacro)
@@ -276,5 +276,5 @@
       </inertial>
       <visual>
-        <origin xyz="0 0 0" rpy="0 3.14159 0"/>
+        <origin xyz="0 0 0" rpy="3.14159 3.14159 0"/>
         <geometry>
           <mesh filename="package://abb_irb120_support/meshes/irb120_3_58/visual/link_5.stl"/>
@@ -283,5 +283,5 @@
       </visual>
       <collision>
-        <origin xyz="0 0 0" rpy="0 3.14159 0"/>
+        <origin xyz="0 0 0" rpy="3.14159 3.14159 0"/>
         <geometry>
           <mesh filename="package://abb_irb120_support/meshes/irb120_3_58/collision/link_5.stl"/>
